File: tokyo.brd (EAGLE design)
At the start: 115 x 34 mm, 47 parts, among them J1 254-2X5F, J2 254-2X5M, P1 9774050151, P2 9774050151, P3 9774050151, P4 9774050151, Q1 BUL7216, T1 750313823, U1 TCLD1000, U2 UCC28720, X1 508-1X3B

Commit message: Ready for manufacture.
Parts:
- removed U2: UCC28720, integratedcircuits:SOIC7
- added C13, C14: 2200p/250V, capacitors:2211
- added D8: SMCJ400CA, supressors:DO-214AB
- added R12, R13: 332k, resistors:1206
- added TP1: TESTPOINT, unsorted:TESTPOINT
- C10: value 4.7u/50v -> 1n/2kV; device capacitors:1206 -> capacitors:1812
- C11: value 2200p/250V -> 10u/50v; device capacitors:2211 -> capacitors:1206
- C12: value 2200p/250V -> 100n; device capacitors:2211 -> capacitors:0603
- C4, C5: value 2200u -> 1800u; device capacitors:D10 -> capacitors:D13
- C7: value 1n/2kv -> 1n/2kV
- C8: value 1n/2kV -> 22u; device capacitors:1812 -> capacitors:1206
- C9: value 1n/2kV -> 1n/2kv
- D2: value PDS1040L -> BAS21; device diodes:POWERDI5 -> diodes:SOT23
- D3: value SMBJ85A -> PDS1040L; device supressors:DO-214AA -> diodes:POWERDI5
- D4: value DFLR1600 -> SMBJ85A; device diodes:POWERDI123 -> supressors:DO-214AA
- D5: value BAS21 -> MURS360S; device diodes:SOT23 -> diodes:DO-214AA
- D6: value HD06 -> BAS21; device diodes:MINIDIP -> diodes:SOT23
- D7: value SMCJ400CA -> HD06; device supressors:DO-214AB -> diodes:MINIDIP
- Q1: value BUL7216 -> STD6N95K5; device transistors:TO220V -> transistors:DPAK
- R10: value 332k -> 1k; device resistors:1206 -> resistors:0603
- R11: value 332k -> 0.5; device resistors:1206 -> resistors:2512
- R2: value 4k87 -> 1k
- R4: value 1.96k -> 130; device resistors:0603 -> resistors:1206
- R5: value 130 -> 39; device resistors:1206 -> resistors:0603
- R6: value 1 -> 121k; device resistors:2512 -> resistors:0603
- R7: value 4k87 -> 24k9
- R8: value 120k -> 10k
- R9: value 24k9 -> 10
- U1: value TCLD1000 -> UCC28710; device unsorted:SOP-4L -> integratedcircuits:SOIC7
- moved C9 36.7 mm to (82.9, 14.3)
- moved C12 36.5 mm to (45.6, 11.2), turned to 90 degrees
- moved C11 35.0 mm to (47.7, 10.8), turned to 90 degrees
- moved D6 29.1 mm to (52.2, 9.89), turned to 0 degrees
- moved R2 27.7 mm to (108.0, 21.8)
- moved D3 27.1 mm to (78.0, 16.8), turned to 270 degrees
- moved LD1 25.1 mm to (107.6, 23.7), turned to 180 degrees
- moved D5 24.1 mm to (58.2, 27.1), turned to 180 degrees
- moved U1 24.1 mm to (40.7, 8.48), turned to 0 degrees
- moved C10 21.3 mm to (61.7, 16.9), turned to 0 degrees
- moved R4 20.2 mm to (63.5, 25.9), turned to 270 degrees
- moved C8 20.0 mm to (84.0, 22.3), turned to 90 degrees
- moved D4 18.8 mm to (61.8, 21.2), turned to 180 degrees
- moved R5 15.9 mm to (49.8, 9.97), turned to 90 degrees
- moved C7 13.4 mm to (86.1, 3.26), turned to 270 degrees
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Connections:
- removed net N$24: R4.2, U1.1
- removed net N$25: D1.1, RL1.16, U1.4
- new net N$23: R9.1, U1.6
- new net N$26: D6.3, R5.2
- new net N$27: C8.1, D1.3, D2.3, RL1.1
- net +5V/1: now also C9.2, D3.P$3; no longer C7.2, D1.3, D2.P$3, RL1.1
- net 0V: now also C11.2, C12.2, D7.2, R11.1, R12.2, R7.2, R8.1, TP1.P$1, U1.4; no longer C10.2, D6.2, R10.2, R6.1, R9.2, U1.2, U2.4
- net 0V/1: now also C7.1, C8.2, D1.1, RL1.16; no longer C8.1, U1.3
- net EARTH: now also C13.2, C14.1, C7.2; no longer C11.2, C12.1, C8.2
- net N$1: now also C14.2; no longer C12.2
- net N$10: now also D5.2, R4.1; no longer D4.2, R5.1
- net N$11: now also C10.2, D4.1; no longer C9.2, D3.1
- net N$12: now also R10.2, R11.2; no longer R6.2, R7.2
- net N$13: now also R10.1, U1.5; no longer R7.1, U2.5
- net N$14: now also R8.2, R9.2; no longer U2.6
- net N$15: now also C11.1, C12.1, R5.1, U1.1; no longer C10.1, D5.3, R4.1, U2.1
- net N$16: now also R12.1, R13.2; no longer R10.1, R11.2
- net N$17: now also C10.1, D4.2, R4.2; no longer C9.1, D3.2, R5.2
- net N$18: now also R6.2, R7.1, U1.2; no longer R8.2, R9.1, U2.2
- net N$2: now also C13.1, D7.4, D8.P$1; no longer C11.1, D6.4, D7.P$1
- net N$3: now also D6.1, R6.1; no longer D5.1, R8.1
- net N$4: now also D7.3, D8.P$2; no longer D6.3, D7.P$2
- net N$6: now also C9.1; no longer C7.1
- net N$7: now also D7.1, R13.1; no longer D6.1, R11.1
- net N$8: now also D2.1, D3.P$1, D3.P$2; no longer D2.P$1, D2.P$2
- net N$9: now also D5.1, U1.8; no longer D4.1, U2.8
Routing:
- net N$11: track 21.0 -> 88.0 mm, vias 0 -> 26
- net N$25: track 45.2 -> 0.00 mm, vias 1 -> 0
- net N$27: track 0.00 -> 38.4 mm, vias 0 -> 1
- net 0V/1: track 90.7 -> 72.1 mm
- net N$15: track 25.5 -> 6.96 mm, vias 2 -> 0
- net N$3: track 25.7 -> 8.47 mm, vias 1 -> 0
- net N$14: track 17.9 -> 3.81 mm
- net 0V: track 96.4 -> 109.8 mm, vias 2 -> 0
- net N$9: track 33.1 -> 45.5 mm, vias 0 -> 1
- net +5V/1: track 67.5 -> 55.2 mm
- net N$23: track 0.00 -> 7.68 mm
- net N$13: track 8.70 -> 2.60 mm
- net N$19: track 19.4 -> 23.7 mm
- net N$8: track 10.2 -> 12.9 mm
- net +5V/2: track 16.6 -> 13.9 mm
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- added copper zone on layer 16, net 0V
- added copper zone on layer 1, net N$11
- added copper zone on layer 16, net N$11
- added copper zone on layer 16, net N$24
- removed copper zone on layer 1, net N$20
