File: tokyo.sch (EAGLE design)
At the start: 47 parts, among them J1 254-2X5F, J2 254-2X5M, P1 9774050151, P2 9774050151, P3 9774050151, P4 9774050151, Q1 BUL7216, T1 750313823, U1 TCLD1000, U2 UCC28720, X1 508-1X3B

Commit message: Ready for manufacture.
Parts:
- removed U2: UCC28720, integratedcircuits:UCC28720
- added C13, C14: 2200p/250V, capacitors:C2211
- added D8: SMCJ400CA, supressors:SMCJ400CA
- added R12, R13: 332k, resistors:R1206
- added TP1: TESTPOINT, unsorted:TESTPOINT
- C10: value 4.7u/50v -> 1n/2kV; device capacitors:C1206 -> capacitors:C1812
- C11: value 2200p/250V -> 10u/50v; device capacitors:C2211 -> capacitors:C1206
- C12: value 2200p/250V -> 100n; device capacitors:C2211 -> capacitors:C0603
- C4, C5: value 2200u -> 1800u; device capacitors:C+D10 -> capacitors:C+D13
- C7: value 1n/2kv -> 1n/2kV
- C8: value 1n/2kV -> 22u; device capacitors:C1812 -> capacitors:C1206
- C9: value 1n/2kV -> 1n/2kv
- D2: value PDS1040L -> BAS21; device diodes:PDS1040L -> diodes:BAS21
- D3: value SMBJ85A -> PDS1040L; device supressors:SMBJ85A -> diodes:PDS1040L
- D4: value DFLR1600 -> SMBJ85A; device diodes:DFLR1600 -> supressors:SMBJ85A
- D5: value BAS21 -> MURS360S; device diodes:BAS21 -> diodes:MURS360S
- D6: value HD06 -> BAS21; device diodes:HD06 -> diodes:BAS21
- D7: value SMCJ400CA -> HD06; device supressors:SMCJ400CA -> diodes:HD06
- Q1: value BUL7216 -> STD6N95K5; device transistors:BUL7216 -> transistors:STD6N95K5
- R10: value 332k -> 1k; device resistors:R1206 -> resistors:R0603
- R11: value 332k -> 0.5; device resistors:R1206 -> resistors:R2512
- R2: value 4k87 -> 1k
- R4: value 1.96k -> 130; device resistors:R0603 -> resistors:R1206
- R5: value 130 -> 39; device resistors:R1206 -> resistors:R0603
- R6: value 1 -> 121k; device resistors:R2512 -> resistors:R0603
- R7: value 4k87 -> 24k9
- R8: value 120k -> 10k
- R9: value 24k9 -> 10
- U1: value TCLD1000 -> UCC28710; device unsorted:TCLD1000 -> integratedcircuits:UCC28710
Connections:
- removed net N$24: R4.2, U1.1
- removed net N$25: D1.2, RL1G$1.2, U1.4
- new net N$23: R9.1, U1.DRV
- new net N$26: D6.1, R5.2
- new net N$27: C8.1, D1.1, D2.1, RL1G$1.1
- net +5V/1: now also C9.2, D3.1; no longer C7.2, D1.1, D2.1, RL1G$1.1
- net 0V: now also C11.2, C12.2, D7.2, R11.1, R12.2, R7.2, R8.1, TP1.P$1, U1.GND; no longer C10.2, D6.2, R10.2, R6.1, R9.2, U1.2, U2.GND
- net 0V/1: now also C7.1, C8.2, D1.2, RL1G$1.2; no longer C8.1, U1.3
- net EARTH: now also C13.1, C14.2, C7.2; no longer C11.1, C12.2, C8.2
- net N$1: now also C14.1; no longer C12.1
- net N$10: now also D5.2, R4.1; no longer D4.2, R5.1
- net N$11: now also C10.2, D4.C, Q1.D; no longer C9.2, D3.C, Q1.C
- net N$12: now also Q1.S, R10.2, R11.2; no longer Q1.E, R6.2, R7.2
- net N$13: now also R10.1, U1.CS; no longer R7.1, U2.CS
- net N$14: now also Q1.G, R8.2, R9.2; no longer Q1.B, U2.DRV
- net N$15: now also C11.1, C12.1, R5.1, U1.VDD; no longer C10.1, D5.1, R4.1, U2.VDD
- net N$16: now also R12.1, R13.2; no longer R10.1, R11.2
- net N$17: now also C10.1, D4.A, R4.2; no longer C9.1, D3.A, R5.2
- net N$18: now also R6.2, R7.1, U1.VS; no longer R8.2, R9.1, U2.VS
- net N$2: now also C13.2, D7.4, D8.P$1; no longer C11.2, D6.4, D7.P$1
- net N$3: now also D6.2, R6.1; no longer D5.2, R8.1
- net N$4: now also D7.3, D8.P$2; no longer D6.3, D7.P$2
- net N$6: now also C9.1; no longer C7.1
- net N$7: now also D7.1, R13.1; no longer D6.1, R11.1
- net N$8: now also D3.2
- net N$9: now also D5.1, U1.HV; no longer D4.1, U2.HV
Other:
- moved on the sheet: C10, C11, C12, C2, C3, C7, C8, C9, D1, D2, D5, L1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
